File: hardware_v1/im483i_daughter/motion_daughter.brd (EAGLE design)
At the start: 70 x 70 mm, 12 parts, among them J1 WW-34P-SPECIALIM483I_HEADER, J2 WW-10P5

Commit message: hardware_v1: change resistor values, add pdfs
Parts:
- R1, R3, R5: value 220 -> 970
- R2, R4: value 47 -> 470
Changed lines of the file:
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@@
 <?xml version="1.0" encoding="utf-8"?>
 <!DOCTYPE eagle SYSTEM "eagle.dtd">
-<eagle version="7.6.0">
+<eagle version="7.7.0">
 <drawing>
 <settings>
@@
 <attribute name="VALUE" x="14.209" y="6.415" size="1.27" layer="27" ratio="10" rot="R270"/>
 </element>
-<element name="R1" library="resistor" package="0207/7" value="220" x="33.56" y="61.82"/>
-<element name="R2" library="resistor" package="0207/7" value="47" x="33.56" y="55.2"/>
-<element name="R3" library="resistor" package="0207/7" value="220" x="33.56" y="48.58"/>
-<element name="R4" library="resistor" package="0207/7" value="47" x="33.56" y="14.94"/>
-<element name="R5" library="resistor" package="0207/7" value="220" x="33.56" y="8.32"/>
+<element name="R1" library="resistor" package="0207/7" value="970" x="33.56" y="61.82"/>
+<element name="R2" library="resistor" package="0207/7" value="470" x="33.56" y="55.2"/>
+<element name="R3" library="resistor" package="0207/7" value="970" x="33.56" y="48.58"/>
+<element name="R4" library="resistor" package="0207/7" value="470" x="33.56" y="14.94"/>
+<element name="R5" library="resistor" package="0207/7" value="970" x="33.56" y="8.32"/>
 </elements>
 <signals>
