File: hardware_v1/im483i_daughter/motion_daughter.sch (EAGLE design)
At the start: 12 parts, among them J1 WW-34P-SPECIALIM483I_HEADER, J2 WW-10P5

Commit message: hardware_v1: change resistor values, add pdfs
Parts:
- R1, R3, R5: value 220 -> 970
- R2, R4: value 47 -> 470
Changed lines of the file:
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@@
 <?xml version="1.0" encoding="utf-8"?>
 <!DOCTYPE eagle SYSTEM "eagle.dtd">
-<eagle version="7.6.0">
+<eagle version="7.7.0">
 <drawing>
 <settings>
@@
 <part name="MOVE" library="led" deviceset="LED" device="3MM"/>
 <part name="FAULT" library="led" deviceset="LED" device="3MM"/>
-<part name="R1" library="resistor" deviceset="R-US_" device="0207/7" value="220"/>
-<part name="R2" library="resistor" deviceset="R-US_" device="0207/7" value="47"/>
-<part name="R3" library="resistor" deviceset="R-US_" device="0207/7" value="220"/>
-<part name="R4" library="resistor" deviceset="R-US_" device="0207/7" value="47"/>
-<part name="R5" library="resistor" deviceset="R-US_" device="0207/7" value="220"/>
+<part name="R1" library="resistor" deviceset="R-US_" device="0207/7" value="970"/>
+<part name="R2" library="resistor" deviceset="R-US_" device="0207/7" value="470"/>
+<part name="R3" library="resistor" deviceset="R-US_" device="0207/7" value="970"/>
+<part name="R4" library="resistor" deviceset="R-US_" device="0207/7" value="470"/>
+<part name="R5" library="resistor" deviceset="R-US_" device="0207/7" value="970"/>
 <part name="SUPPLY1" library="supply2" deviceset="VCC" device=""/>
 <part name="SUPPLY2" library="supply2" deviceset="VCC" device=""/>
